File: design/sch-pcb/proj/proj.kicad_sch (KiCad schematic)
At the start: 9 parts

Commit message: algo
cambie algunas cosas
Parts:
- removed C3: C, symbol Device:C
- removed R4, R5: R, symbol Device:R
- added SW1, SW2, SW3: SW_Push_Open_Dual_x2, symbol Switch:SW_Push_Open_Dual_x2
Connections:
- net +3.3V: now also R1.1, R2.1, R3.1
- net GPIO: now reaches C2.1
- net GPIO: now also C1.1, C4.1, R1.2, R2.2, R3.2, SW1.1, SW2.1, SW3.1
- net GND: now reaches C2.2
- net GND: now also C1.2, C4.2, SW1.2, SW2.2, SW3.2
Other:
- moved on the sheet: C1, C2, C4, R1, R2
